Commit message: Sim turn-rate calibration on the cave floor, and keep the Spin recovery
- explorer_gazebo.xacro: skid_track 0.43 -> 0.34. Against Gazebo's true pose the robot turned
  1.2-1.3x the commanded yaw rate on the cave floor (all command sizes, 0.15-0.25 s delay
  allowed); the EKF heading matched the truth exactly. MPPI assumes commands are achieved, so it
  swung past the path heading (+65 deg) and needed 300-450 deg of turning to settle.
  0.43 / 1.25 = 0.34 gives 0.98x in a check run. The real robot's track_width is unchanged.
- explore_nav_to_pose_demo.xml: Spin restored. Without it, MPPI deadlocks facing a wall in dead
  ends had no way out (stuck time 7 % -> 31 %, goal success 59 % -> 35 % in 3 GUI runs), and
  the >= 300 deg rotation events did not drop.

Co-Authored-By: Claude Opus 5.5 <noreply@anthropic.com>

File: src/explorer_description/urdf/explorer_gazebo.xacro (robot description, xacro)
@@ -10,5 +10,11 @@
     </gazebo>
   </xacro:macro>
-  <xacro:property name="skid_track" value="0.43"/>
+  <!-- Effective skid-steer track for Gazebo's DiffDrive (exp/tunnel-tracking, 2026-10-19: was 0.43).
+       0.43 was calibrated turning on the spot in empty.sdf (0.90-1.08x of the command). On the
+       cave floor the robot turned 1.2-1.3x the commanded yaw rate (Gazebo true pose, 4 GUI runs,
+       all command sizes, 0.15-0.25 s delay allowed), so MPPI swung past the path heading and
+       turned 300+ deg to settle. 0.43 / 1.25 = 0.34. The real robot keeps its own value
+       (explorer_bringup track_width). -->
+  <xacro:property name="skid_track" value="0.34"/>
   <xacro:wheel_grip name="left_front"/>
   <xacro:wheel_grip name="left_middle"/>

Commit message: Ablation set-up: one change of the demo config undone per variant
Version under test: tag nav-demo-v2 (exp/tunnel-tracking). Stuck time rose from 7 % (tuned) to
33 % with the demo fixes. Each variant undoes exactly one of the four differences:
A config/nav2_params_abl_unknown.yaml  : allow_unknown true, global costmap on /map
B config/nav2_params_abl_handover.yaml : GoalCritic / PathFollowCritic hand-over at 1.0 m
C skid_track:=0.43                     : sim track width (new launch argument, default 0.34)
D precheck_path:=false                 : no planner pre-check in the coordinator

Co-Authored-By: Claude Opus 5.5 <noreply@anthropic.com>

File: src/explorer_description/urdf/explorer_gazebo.xacro (robot description, xacro)
@@ -16,5 +16,6 @@
        turned 300+ deg to settle. 0.43 / 1.25 = 0.34. The real robot keeps its own value
        (explorer_bringup track_width). -->
-  <xacro:property name="skid_track" value="0.34"/>
+  <xacro:arg name="skid_track" default="0.34"/>   <!-- launch argument, for the 2026-10-20 ablation -->
+  <xacro:property name="skid_track" value="$(arg skid_track)"/>
   <xacro:wheel_grip name="left_front"/>
   <xacro:wheel_grip name="left_middle"/>
